File: SE_placa/cargador_regulador.sch (KiCad schematic (older format))
At the start: 17 parts, among them IC1 TP4056, U3 LTC3441EDEPBF

Commit message: Actualizacion PCB
Organizo archivos, agrego nuevos elementos a footprint, actualizo net list y actualizo PCB, agrego modelos 3D disponibles. Listo para iniciar ruteo
Parts:
- C10, C11, C12, C13, C9: footprint (none) -> Capacitor_SMD:C_0805_2012Metric_Pad1.18x1.45mm_HandSolder
- D6, D7: footprint (none) -> LED_SMD:LED_0805_2012Metric_Pad1.15x1.40mm_HandSolder
- IC1: footprint SOP-8 -> TP4056:SOP-8; symbol TP4056:TP4056 -> SE_placa-rescue:TP4056-TP4056
- L4: footprint (none) -> 1264EY-4R7M_P3:IND_1264EY-4R7M=P3
- R19, R20, R21, R22, R23, R24, R25: footprint (none) -> Resistor_SMD:R_0805_2012Metric_Pad1.20x1.40mm_HandSolder
- U3: footprint DFN400X300X80-13N -> LTC3441EDEPBF:DFN400X300X80-13N
Changed lines of the file:
@@
 F 0 "C10" H 5040 2946 50  0000 L CNN
 F 1 "10uF" H 5040 2855 50  0000 L CNN
-F 2 "" H 4963 2750 50  0001 C CNN
+F 2 "Capacitor_SMD:C_0805_2012Metric_Pad1.18x1.45mm_HandSolder" H 4963 2750 50  0001 C CNN
 F 3 "~" H 4925 2900 50  0001 C CNN
 	1    4925 2900
@@
 F 0 "D6" H 2418 2720 50  0000 C CNN
 F 1 "LED" H 2418 2811 50  0000 C CNN
-F 2 "" H 2425 2975 50  0001 C CNN
+F 2 "LED_SMD:LED_0805_2012Metric_Pad1.15x1.40mm_HandSolder" H 2425 2975 50  0001 C CNN
 F 3 "~" H 2425 2975 50  0001 C CNN
 	1    2425 2975
@@
 F 0 "D7" H 2443 3145 50  0000 C CNN
 F 1 "LED" H 2443 3236 50  0000 C CNN
-F 2 "" H 2450 3400 50  0001 C CNN
+F 2 "LED_SMD:LED_0805_2012Metric_Pad1.15x1.40mm_HandSolder" H 2450 3400 50  0001 C CNN
 F 3 "~" H 2450 3400 50  0001 C CNN
 	1    2450 3400
@@
 F 0 "R19" H 2070 2396 50  0000 L CNN
 F 1 "0.4 ohm" H 2070 2305 50  0000 L CNN
-F 2 "" V 1930 2350 50  0001 C CNN
+F 2 "Resistor_SMD:R_0805_2012Metric_Pad1.20x1.40mm_HandSolder" V 1930 2350 50  0001 C CNN
 F 3 "~" H 2000 2350 50  0001 C CNN
 	1    2000 2350
@@
 $EndComp
 $Comp
-L TP4056:TP4056 IC?
+L SE_placa-rescue:TP4056-TP4056 IC?
 U 1 1 60A44197
 P 3800 2975
@@
 F 0 "IC1" H 3800 3542 50  0000 C CNN
 F 1 "TP4056" H 3800 3451 50  0000 C CNN
-F 2 "SOP-8" H 3800 2975 50  0001 L BNN
+F 2 "TP4056:SOP-8" H 3800 2975 50  0001 L BNN
 F 3 "" H 3800 2975 50  0001 L BNN
 	1    3800 2975
@@
 F 0 "C9" H 1540 3021 50  0000 L CNN
 F 1 "10uF" H 1540 2930 50  0000 L CNN
-F 2 "" H 1463 2825 50  0001 C CNN
+F 2 "Capacitor_SMD:C_0805_2012Metric_Pad1.18x1.45mm_HandSolder" H 1463 2825 50  0001 C CNN
 F 3 "~" H 1425 2975 50  0001 C CNN
 	1    1425 2975
@@
 F 0 "R22" H 4570 3421 50  0000 L CNN
 F 1 "8.2K" H 4570 3330 50  0000 L CNN
-F 2 "" V 4430 3375 50  0001 C CNN
+F 2 "Resistor_SMD:R_0805_2012Metric_Pad1.20x1.40mm_HandSolder" V 4430 3375 50  0001 C CNN
 F 3 "~" H 4500 3375 50  0001 C CNN
 	1    4500 3375
@@
 F 0 "U3" H 7375 3945 50  0000 C CNN
 F 1 "LTC3441EDEPBF" H 7375 3854 50  0000 C CNN
-F 2 "DFN400X300X80-13N" H 7375 2975 50  0001 L BNN
+F 2 "LTC3441EDEPBF:DFN400X300X80-13N" H 7375 2975 50  0001 L BNN
 F 3 "" H 7375 2975 50  0001 L BNN
 F 4 "Linear Technology" H 7375 2975 50  0001 L BNN "SUPPLIER"
@@
 F 0 "C11" H 5565 2946 50  0000 L CNN
 F 1 "10uF" H 5565 2855 50  0000 L CNN
-F 2 "" H 5488 2750 50  0001 C CNN
+F 2 "Capacitor_SMD:C_0805_2012Metric_Pad1.18x1.45mm_HandSolder" H 5488 2750 50  0001 C CNN
 F 3 "~" H 5450 2900 50  0001 C CNN
 	1    5450 2900
@@
 F 0 "R23" V 8168 2875 50  0000 C CNN
 F 1 "15K" V 8259 2875 50  0000 C CNN
-F 2 "" V 8305 2875 50  0001 C CNN
+F 2 "Resistor_SMD:R_0805_2012Metric_Pad1.20x1.40mm_HandSolder" V 8305 2875 50  0001 C CNN
 F 3 "~" H 8375 2875 50  0001 C CNN
 	1    8375 2875
@@
 F 0 "C12" H 8915 2921 50  0000 L CNN
 F 1 "1.5nF" H 8915 2830 50  0000 L CNN
-F 2 "" H 8838 2725 50  0001 C CNN
+F 2 "Capacitor_SMD:C_0805_2012Metric_Pad1.18x1.45mm_HandSolder" H 8838 2725 50  0001 C CNN
 F 3 "~" H 8800 2875 50  0001 C CNN
 	1    8800 2875
@@
 F 0 "R25" H 9305 3254 50  0000 R CNN
 F 1 "200K" H 9305 3345 50  0000 R CNN
-F 2 "" V 9305 3300 50  0001 C CNN
+F 2 "Resistor_SMD:R_0805_2012Metric_Pad1.20x1.40mm_HandSolder" V 9305 3300 50  0001 C CNN
 F 3 "~" H 9375 3300 50  0001 C CNN
 	1    9375 3300
@@
 F 0 "R24" H 9305 2579 50  0000 R CNN
 F 1 "340K" H 9305 2670 50  0000 R CNN
-F 2 "" V 9305 2625 50  0001 C CNN
+F 2 "Resistor_SMD:R_0805_2012Metric_Pad1.20x1.40mm_HandSolder" V 9305 2625 50  0001 C CNN
 F 3 "~" H 9375 2625 50  0001 C CNN
 	1    9375 2625
@@
 F 0 "C13" H 10090 2996 50  0000 L CNN
 F 1 "22uF" H 10090 2905 50  0000 L CNN
-F 2 "" H 10013 2800 50  0001 C CNN
+F 2 "Capacitor_SMD:C_0805_2012Metric_Pad1.18x1.45mm_HandSolder" H 10013 2800 50  0001 C CNN
 F 3 "~" H 9975 2950 50  0001 C CNN
 	1    9975 2950
@@
 F 0 "L4" V 6390 2975 50  0000 C CNN
 F 1 "4.7 uH" V 6299 2975 50  0000 C CNN
-F 2 "" H 6200 2975 50  0001 C CNN
-F 3 "~" H 6200 2975 50  0001 C CNN
+F 2 "1264EY-4R7M_P3:IND_1264EY-4R7M=P3" H 6200 2975 50  0001 C CNN
+F 3 "~http://www.farnell.com/datasheets/2616901.pdf" H 6200 2975 50  0001 C CNN
 	1    6200 2975
 	0    -1   -1   0
@@
 F 0 "R20" V 2693 2975 50  0000 C CNN
 F 1 "2K" V 2784 2975 50  0000 C CNN
-F 2 "" V 2830 2975 50  0001 C CNN
+F 2 "Resistor_SMD:R_0805_2012Metric_Pad1.20x1.40mm_HandSolder" V 2830 2975 50  0001 C CNN
 F 3 "~" H 2900 2975 50  0001 C CNN
 	1    2900 2975
@@
 F 0 "R21" V 2718 3400 50  0000 C CNN
 F 1 "2K" V 2809 3400 50  0000 C CNN
-F 2 "" V 2855 3400 50  0001 C CNN
+F 2 "Resistor_SMD:R_0805_2012Metric_Pad1.20x1.40mm_HandSolder" V 2855 3400 50  0001 C CNN
 F 3 "~" H 2925 3400 50  0001 C CNN
 	1    2925 3400

Commit message: Ubicaciones de librerias de absolutas a relativas
Parts:
- U3: symbol LTC3441EDEPBF:LTC3441EDEPBF -> SE_placa-rescue:LTC3441EDEPBF-LTC3441EDEPBF
Changed lines of the file:
@@
 	4750 2075 4925 2075
 $Comp
-L LTC3441EDEPBF:LTC3441EDEPBF U3
+L SE_placa-rescue:LTC3441EDEPBF-LTC3441EDEPBF U3
 U 1 1 609461A1
 P 7375 2975
+AR Path="/609461A1" Ref="U3"  Part="1"
+AR Path="/609FB393/609461A1" Ref="U3"  Part="1"
 F 0 "U3" H 7375 3945 50  0000 C CNN
 F 1 "LTC3441EDEPBF" H 7375 3854 50  0000 C CNN

Commit message: Ruteo 3
1. Cambio orden de los pines de I/O para hacer mas facil el ruteo de los conectores, modifico ubicacion de I/Os del Lora
2. Cambio huella del LTC 3441 al parecer la que tenia creaba conflictos con las rutas y sus anchos
3. cambio el esquema de Net classes a default, arreglando el tamaño de las rutas y de las vias .
4. Modifico la ruta a 0.3 mm , agrego esto a pre definidas
5. agrego ruta de 1 mm y vias de 1.8 mm para alimentaciones
6. cambio ubicaciones de conectorres de bateria y de panel solar
7. cambio ubicacion del TP4056 y modifico la ubicacion de los componentes cercanos.
8. Falta agregar plano de tierra en las dos caras y modificar salida de potencia de la entrada y la salida del LTC 3441
Parts:
- U3: footprint LTC3441EDEPBF:DFN400X300X80-13N -> LTC3441EDE#PBF:SON50P300X400X80-13N-D
Changed lines of the file:
@@
 F 0 "U3" H 7375 3945 50  0000 C CNN
 F 1 "LTC3441EDEPBF" H 7375 3854 50  0000 C CNN
-F 2 "LTC3441EDEPBF:DFN400X300X80-13N" H 7375 2975 50  0001 L BNN
+F 2 "LTC3441EDE#PBF:SON50P300X400X80-13N-D" H 7375 2975 50  0001 L BNN
 F 3 "" H 7375 2975 50  0001 L BNN
 F 4 "Linear Technology" H 7375 2975 50  0001 L BNN "SUPPLIER"
